Commit message: adjust controller and initial position

File: burke_description/urdf/components/ur8long.urdf.xacro (robot description, xacro)
@@ -12,7 +12,10 @@
       physical_parameters_file
       visual_parameters_file">
-    <!-- Simulation tuning: moderate viscous joint damping prevents gravity
-         oscillation without making the arm sluggish. Units are N*m*s/rad. -->
-    <xacro:property name="arm_joint_damping" value="0.5"/>
+    <!-- Simulation tuning: the geared UR joints have appreciable effective
+         damping. Use more damping on the load-bearing joints and less on the
+         lightweight wrist joints. Units are N*m*s/rad. -->
+    <xacro:property name="shoulder_joint_damping" value="20.0"/>
+    <xacro:property name="elbow_joint_damping" value="10.0"/>
+    <xacro:property name="wrist_joint_damping" value="2.0"/>
     <!-- Small Coulomb friction reduces gravity-driven drift at rest. Units are
          N*m. This remains intentionally lower than the damping contribution. -->
@@ -104,5 +107,5 @@
       <xacro:official_inertial key="wrist_3" mass_key="wrist_3_mass" cog_key="wrist_3_cog"/>
     </link>
-    <xacro:macro name="ur_joint" params="name parent child kinematics_key limits_key">
+    <xacro:macro name="ur_joint" params="name parent child kinematics_key limits_key damping">
       <xacro:property name="pose" value="${kinematics_data[kinematics_key]}"/>
       <xacro:property name="limit" value="${limits_data[limits_key]}"/>
@@ -113,13 +116,17 @@
         <axis xyz="0 0 1"/>
         <limit lower="${limit['lower']}" upper="${limit['upper']}" effort="${limit['effort']}" velocity="${limit['velocity']}"/>
-        <dynamics damping="${arm_joint_damping}" friction="${arm_joint_friction}"/>
+        <dynamics damping="${damping}" friction="${arm_joint_friction}"/>
       </joint>
     </xacro:macro>
-    <xacro:ur_joint name="arm_joint_1" parent="arm_mount_link" child="arm_link_1" kinematics_key="shoulder" limits_key="shoulder_pan_joint"/>
-    <xacro:ur_joint name="arm_joint_2" parent="arm_link_1" child="arm_link_2" kinematics_key="upper_arm" limits_key="shoulder_lift_joint"/>
-    <xacro:ur_joint name="arm_joint_3" parent="arm_link_2" child="arm_link_3" kinematics_key="forearm" limits_key="elbow_joint"/>
-    <xacro:ur_joint name="arm_joint_4" parent="arm_link_3" child="arm_link_4" kinematics_key="wrist_1" limits_key="wrist_1_joint"/>
-    <xacro:ur_joint name="arm_joint_5" parent="arm_link_4" child="arm_link_5" kinematics_key="wrist_2" limits_key="wrist_2_joint"/>
-    <xacro:ur_joint name="arm_joint_6" parent="arm_link_5" child="arm_link_6" kinematics_key="wrist_3" limits_key="wrist_3_joint"/>
+    <xacro:ur_joint name="arm_joint_1" parent="arm_mount_link" child="arm_link_1" kinematics_key="shoulder" limits_key="shoulder_pan_joint" damping="${shoulder_joint_damping}"/>
+    <xacro:ur_joint name="arm_joint_2" parent="arm_link_1" child="arm_link_2" kinematics_key="upper_arm" limits_key="shoulder_lift_joint" damping="${shoulder_joint_damping}"/>
+    <xacro:ur_joint name="arm_joint_3" parent="arm_link_2" child="arm_link_3" kinematics_key="forearm" limits_key="elbow_joint" damping="${elbow_joint_damping}"/>
+    <xacro:ur_joint name="arm_joint_4" parent="arm_link_3" child="arm_link_4" kinematics_key="wrist_1" limits_key="wrist_1_joint" damping="${wrist_joint_damping}"/>
+    <xacro:ur_joint name="arm_joint_5" parent="arm_link_4" child="arm_link_5" kinematics_key="wrist_2" limits_key="wrist_2_joint" damping="${wrist_joint_damping}"/>
+    <xacro:ur_joint name="arm_joint_6" parent="arm_link_5" child="arm_link_6" kinematics_key="wrist_3" limits_key="wrist_3_joint" damping="${wrist_joint_damping}"/>
+    <!-- Keep Gazebo's direct position mode, but use conservative simulated
+         actuator speeds instead of stepping at the UR hardware velocity
+         limits. This avoids exciting the coupled links while preserving a
+         stiff final position. -->
     <xacro:macro name="arm_position_controller" params="joint topic speed initial_position">
       <gazebo>
@@ -134,11 +141,11 @@
       </gazebo>
     </xacro:macro>
-    <!-- Default pose in degrees: [0, -90, 0, -90, 0, 0]. -->
-    <xacro:arm_position_controller joint="arm_joint_1" topic="/model/burke_base/arm/joint_1/command" speed="${limits_data['shoulder_pan_joint']['velocity']}" initial_position="0.0"/>
-    <xacro:arm_position_controller joint="arm_joint_2" topic="/model/burke_base/arm/joint_2/command" speed="${limits_data['shoulder_lift_joint']['velocity']}" initial_position="${-pi / 2}"/>
-    <xacro:arm_position_controller joint="arm_joint_3" topic="/model/burke_base/arm/joint_3/command" speed="${limits_data['elbow_joint']['velocity']}" initial_position="0.0"/>
-    <xacro:arm_position_controller joint="arm_joint_4" topic="/model/burke_base/arm/joint_4/command" speed="${limits_data['wrist_1_joint']['velocity']}" initial_position="${-pi / 2}"/>
-    <xacro:arm_position_controller joint="arm_joint_5" topic="/model/burke_base/arm/joint_5/command" speed="${limits_data['wrist_2_joint']['velocity']}" initial_position="0.0"/>
-    <xacro:arm_position_controller joint="arm_joint_6" topic="/model/burke_base/arm/joint_6/command" speed="${limits_data['wrist_3_joint']['velocity']}" initial_position="0.0"/>
+    <!-- Default pose in degrees: [0, -120, 120, -90, 90, 0]. -->
+    <xacro:arm_position_controller joint="arm_joint_1" topic="/model/burke_base/arm/joint_1/command" speed="0.75" initial_position="0.0"/>
+    <xacro:arm_position_controller joint="arm_joint_2" topic="/model/burke_base/arm/joint_2/command" speed="0.75" initial_position="${-2*pi / 3}"/>
+    <xacro:arm_position_controller joint="arm_joint_3" topic="/model/burke_base/arm/joint_3/command" speed="1.0" initial_position="${2*pi / 3}"/>
+    <xacro:arm_position_controller joint="arm_joint_4" topic="/model/burke_base/arm/joint_4/command" speed="1.5" initial_position="${-pi / 2}"/>
+    <xacro:arm_position_controller joint="arm_joint_5" topic="/model/burke_base/arm/joint_5/command" speed="1.5" initial_position="${pi / 2}"/>
+    <xacro:arm_position_controller joint="arm_joint_6" topic="/model/burke_base/arm/joint_6/command" speed="1.5" initial_position="0.0"/>
     <gazebo>
       <plugin filename="gz-sim-joint-state-publisher-system" name="gz::sim::systems::JointStatePublisher">
