Commit message: fix joint orientation issue and use real stl

File: burke_description/urdf/burke_base.urdf.xacro (robot description, xacro)
@@ -6,9 +6,27 @@
     values here so Gazebo integration can consume the same values later.
   -->
-  <xacro:property name="chassis_length" value="1.00"/>
-  <xacro:property name="chassis_width" value="0.70"/>
-  <xacro:property name="chassis_height" value="0.22"/>
-  <xacro:property name="chassis_center_z" value="0.23"/>
-  <xacro:property name="chassis_mass" value="45.0"/>
+  <!--
+    CAD visual assumptions from the Task 1 audit:
+    MiR1350_reduced.stl is a reduced 36,106-triangle mesh with measured bounds
+    0.910000 x 1.350000 x 0.321230 m. It is already in metres, so its scale is
+    1.0. The approved yaw is +pi/2, and the mesh origin is retained; its
+    measured bottom is 0.000230 m below the origin.
+  -->
+  <xacro:property name="mir_stl_scale" value="1.0"/>
+  <xacro:property name="mir_visual_length" value="1.350"/>
+  <xacro:property name="mir_visual_width" value="0.910"/>
+  <xacro:property name="mir_visual_height" value="0.321230"/>
+  <xacro:property name="mir_visual_bottom_offset" value="-0.000230"/>
+  <!-- Cancel the small negative STL minimum so the mesh bottom is at base_link. -->
+  <xacro:property name="mir_visual_z_offset" value="${-mir_visual_bottom_offset}"/>
+  <xacro:property name="mir_mesh_yaw" value="${pi / 2}"/>
+  <!-- The 5 mm per-side collision clearance is deliberately conservative. -->
+  <xacro:property name="chassis_length" value="1.340"/>
+  <xacro:property name="chassis_width" value="0.900"/>
+  <xacro:property name="chassis_height" value="0.310963"/>
+  <xacro:property name="chassis_collision_center_z" value="0.1555195"/>
+  <!-- Place base_link and the CAD bottom at the drive-wheel axis height. -->
+  <xacro:property name="chassis_center_z" value="0.120230"/>
+  <xacro:property name="chassis_mass" value="450.0"/>
   <xacro:property name="wheel_radius" value="0.12"/>
   <xacro:property name="wheel_width" value="0.06"/>
@@ -28,4 +46,6 @@
   <xacro:property name="odom_publish_frequency" value="50.0"/>
   <material name="chassis_blue"><color rgba="0.08 0.22 0.42 1.0"/></material>
+  <material name="mir_gray"><color rgba="0.48 0.50 0.53 1.0"/></material>
+  <material name="arm_gray"><color rgba="0.72 0.74 0.77 1.0"/></material>
   <material name="wheel_black"><color rgba="0.03 0.03 0.03 1.0"/></material>
   <material name="caster_gray"><color rgba="0.35 0.35 0.35 1.0"/></material>
@@ -33,18 +53,29 @@
   <link name="base_link">
     <visual>
-      <origin xyz="0 0 0"/>
-      <geometry><box size="${chassis_length} ${chassis_width} ${chassis_height}"/></geometry>
-      <material name="chassis_blue"/>
+      <origin xyz="0 0 ${mir_visual_z_offset}" rpy="0 0 ${mir_mesh_yaw}"/>
+      <geometry>
+        <!-- The reduced mesh is already in metres. -->
+        <mesh filename="package://burke_description/cad/stl/MiR1350_reduced.stl"
+              scale="${mir_stl_scale} ${mir_stl_scale} ${mir_stl_scale}"/>
+      </geometry>
+      <material name="mir_gray"/>
     </visual>
     <collision>
-      <origin xyz="0 0 0"/>
+      <origin xyz="0 0 ${chassis_collision_center_z}"/>
       <geometry><box size="${chassis_length} ${chassis_width} ${chassis_height}"/></geometry>
     </collision>
     <inertial>
-      <origin xyz="0 0 0"/>
+      <origin xyz="0 0 ${chassis_collision_center_z}"/>
       <mass value="${chassis_mass}"/>
-      <inertia ixx="3.006" ixy="0" ixz="0" iyy="4.506" iyz="0" izz="6.006"/>
+      <!-- Solid-box inertia for 45 kg and the collision dimensions above. -->
+      <inertia ixx="3.400117" ixy="0" ixz="0" iyy="7.096117" iyz="0" izz="9.771000"/>
     </inertial>
   </link>
+  <!-- Explicitly retain shadow casting for the CAD visual. -->
+  <gazebo reference="base_link">
+    <visual>
+      <cast_shadows>true</cast_shadows>
+    </visual>
+  </gazebo>
   <joint name="base_footprint_joint" type="fixed">
     <parent link="base_footprint"/>
@@ -54,9 +85,4 @@
   <xacro:macro name="drive_wheel" params="side y">
     <link name="${side}_drive_wheel_link">
-      <visual>
-        <origin rpy="${pi/2} 0 0"/>
-        <geometry><cylinder radius="${wheel_radius}" length="${wheel_width}"/></geometry>
-        <material name="wheel_black"/>
-      </visual>
       <collision>
         <origin rpy="${pi/2} 0 0"/>
@@ -84,5 +110,4 @@
   <xacro:macro name="support_caster" params="name x">
     <link name="${name}_support_link">
-      <visual><geometry><sphere radius="${caster_radius}"/></geometry><material name="caster_gray"/></visual>
       <collision><geometry><sphere radius="${caster_radius}"/></geometry></collision>
       <inertial>
@@ -100,5 +125,5 @@
   <xacro:support_caster name="rear" x="-0.38"/>
   <xacro:ur8long_arm
-    chassis_height="${chassis_height}"
+    arm_mount_z="${mir_visual_height}"
     kinematics_parameters_file="$(find burke_description)/config/ur8long/default_kinematics.yaml"
     joint_limits_parameters_file="$(find burke_description)/config/ur8long/joint_limits.yaml"

File: burke_description/urdf/components/ur8long.urdf.xacro (robot description, xacro)
@@ -7,9 +7,15 @@
   -->
   <xacro:macro name="ur8long_arm" params="
-      chassis_height
+      arm_mount_z
       kinematics_parameters_file
       joint_limits_parameters_file
       physical_parameters_file
       visual_parameters_file">
+    <!-- Simulation tuning: moderate viscous joint damping prevents gravity
+         oscillation without making the arm sluggish. Units are N*m*s/rad. -->
+    <xacro:property name="arm_joint_damping" value="0.5"/>
+    <!-- Small Coulomb friction reduces gravity-driven drift at rest. Units are
+         N*m. This remains intentionally lower than the damping contribution. -->
+    <xacro:property name="arm_joint_friction" value="0.1"/>
     <xacro:property name="kinematics_data" value="${xacro.load_yaml(kinematics_parameters_file)['kinematics']}"/>
     <xacro:property name="limits_data" value="${xacro.load_yaml(joint_limits_parameters_file)['joint_limits']}"/>
@@ -24,4 +30,5 @@
           <mesh filename="package://burke_description/${entry['path']}" scale="${entry['scale']} ${entry['scale']} ${entry['scale']}"/>
         </geometry>
+        <material name="arm_gray"/>
       </visual>
     </xacro:macro>
@@ -64,5 +71,5 @@
       <parent link="base_link"/>
       <child link="arm_mount_link"/>
-      <origin xyz="0 0 ${chassis_height / 2}" rpy="0 0 0"/>
+      <origin xyz="0 0 ${arm_mount_z}" rpy="0 0 0"/>
     </joint>
     <!-- Canonical UR bodies mapped to the stable Burk-e arm_link_N names. -->
@@ -106,5 +113,5 @@
         <axis xyz="0 0 1"/>
         <limit lower="${limit['lower']}" upper="${limit['upper']}" effort="${limit['effort']}" velocity="${limit['velocity']}"/>
-        <dynamics damping="0.0" friction="0.0"/>
+        <dynamics damping="${arm_joint_damping}" friction="${arm_joint_friction}"/>
       </joint>
     </xacro:macro>
@@ -115,10 +122,10 @@
     <xacro:ur_joint name="arm_joint_5" parent="arm_link_4" child="arm_link_5" kinematics_key="wrist_2" limits_key="wrist_2_joint"/>
     <xacro:ur_joint name="arm_joint_6" parent="arm_link_5" child="arm_link_6" kinematics_key="wrist_3" limits_key="wrist_3_joint"/>
-    <xacro:macro name="arm_position_controller" params="joint topic speed">
+    <xacro:macro name="arm_position_controller" params="joint topic speed initial_position">
       <gazebo>
         <plugin filename="gz-sim-joint-position-controller-system" name="gz::sim::systems::JointPositionController">
           <joint_name>${joint}</joint_name>
           <topic>${topic}</topic>
-          <initial_position>0.0</initial_position>
+          <initial_position>${initial_position}</initial_position>
           <use_velocity_commands>true</use_velocity_commands>
           <cmd_max>${speed}</cmd_max>
@@ -127,10 +134,11 @@
       </gazebo>
     </xacro:macro>
-    <xacro:arm_position_controller joint="arm_joint_1" topic="/model/burke_base/arm/joint_1/command" speed="${limits_data['shoulder_pan_joint']['velocity']}"/>
-    <xacro:arm_position_controller joint="arm_joint_2" topic="/model/burke_base/arm/joint_2/command" speed="${limits_data['shoulder_lift_joint']['velocity']}"/>
-    <xacro:arm_position_controller joint="arm_joint_3" topic="/model/burke_base/arm/joint_3/command" speed="${limits_data['elbow_joint']['velocity']}"/>
-    <xacro:arm_position_controller joint="arm_joint_4" topic="/model/burke_base/arm/joint_4/command" speed="${limits_data['wrist_1_joint']['velocity']}"/>
-    <xacro:arm_position_controller joint="arm_joint_5" topic="/model/burke_base/arm/joint_5/command" speed="${limits_data['wrist_2_joint']['velocity']}"/>
-    <xacro:arm_position_controller joint="arm_joint_6" topic="/model/burke_base/arm/joint_6/command" speed="${limits_data['wrist_3_joint']['velocity']}"/>
+    <!-- Default pose in degrees: [0, -90, 0, -90, 0, 0]. -->
+    <xacro:arm_position_controller joint="arm_joint_1" topic="/model/burke_base/arm/joint_1/command" speed="${limits_data['shoulder_pan_joint']['velocity']}" initial_position="0.0"/>
+    <xacro:arm_position_controller joint="arm_joint_2" topic="/model/burke_base/arm/joint_2/command" speed="${limits_data['shoulder_lift_joint']['velocity']}" initial_position="${-pi / 2}"/>
+    <xacro:arm_position_controller joint="arm_joint_3" topic="/model/burke_base/arm/joint_3/command" speed="${limits_data['elbow_joint']['velocity']}" initial_position="0.0"/>
+    <xacro:arm_position_controller joint="arm_joint_4" topic="/model/burke_base/arm/joint_4/command" speed="${limits_data['wrist_1_joint']['velocity']}" initial_position="${-pi / 2}"/>
+    <xacro:arm_position_controller joint="arm_joint_5" topic="/model/burke_base/arm/joint_5/command" speed="${limits_data['wrist_2_joint']['velocity']}" initial_position="0.0"/>
+    <xacro:arm_position_controller joint="arm_joint_6" topic="/model/burke_base/arm/joint_6/command" speed="${limits_data['wrist_3_joint']['velocity']}" initial_position="0.0"/>
     <gazebo>
       <plugin filename="gz-sim-joint-state-publisher-system" name="gz::sim::systems::JointStatePublisher">

Commit message: Integrate liftkit to the simulation

File: burke_description/urdf/burke_base.urdf.xacro (robot description, xacro)
@@ -39,4 +39,5 @@
   <xacro:property name="wheel_mu2" value="0.9"/>
   <xacro:include filename="$(find burke_description)/urdf/components/ur8long.urdf.xacro"/>
+  <xacro:include filename="$(find burke_description)/urdf/components/liftkit.urdf.xacro"/>
   <!-- Simulation assumptions for the bounded base controller. -->
   <xacro:property name="max_linear_velocity" value="0.5"/>
@@ -48,4 +49,5 @@
   <material name="mir_gray"><color rgba="0.48 0.50 0.53 1.0"/></material>
   <material name="arm_gray"><color rgba="0.72 0.74 0.77 1.0"/></material>
+  <material name="liftkit_gray"><color rgba="0.38 0.42 0.47 1.0"/></material>
   <material name="wheel_black"><color rgba="0.03 0.03 0.03 1.0"/></material>
   <material name="caster_gray"><color rgba="0.35 0.35 0.35 1.0"/></material>
@@ -124,6 +126,10 @@
   <xacro:support_caster name="front" x="0.38"/>
   <xacro:support_caster name="rear" x="-0.38"/>
+  <!-- Task 2: add the fixed lower stage and two bounded telescoping stages.
+       The arm remains mounted directly to base_link until Task 3. -->
+  <xacro:liftkit_mast parent_link="base_link" mount_z="${mir_visual_height}"/>
   <xacro:ur8long_arm
-    arm_mount_z="${mir_visual_height}"
+    arm_mount_parent="lift_stage_3_link"
+    arm_mount_z="0.555"
     kinematics_parameters_file="$(find burke_description)/config/ur8long/default_kinematics.yaml"
     joint_limits_parameters_file="$(find burke_description)/config/ur8long/joint_limits.yaml"

File: burke_description/urdf/components/ur8long.urdf.xacro (robot description, xacro)
@@ -7,4 +7,5 @@
   -->
   <xacro:macro name="ur8long_arm" params="
+      arm_mount_parent
       arm_mount_z
       kinematics_parameters_file
@@ -72,5 +73,5 @@
     </link>
     <joint name="arm_mount_joint" type="fixed">
-      <parent link="base_link"/>
+      <parent link="${arm_mount_parent}"/>
       <child link="arm_mount_link"/>
       <origin xyz="0 0 ${arm_mount_z}" rpy="0 0 0"/>

Commit message: fix cad orientation and posisiton

File: burke_description/urdf/burke_base.urdf.xacro (robot description, xacro)
@@ -8,17 +8,12 @@
   <!--
     CAD visual assumptions from the Task 1 audit:
-    MiR1350_reduced.stl is a reduced 36,106-triangle mesh with measured bounds
-    0.910000 x 1.350000 x 0.321230 m. It is already in metres, so its scale is
-    1.0. The approved yaw is +pi/2, and the mesh origin is retained; its
-    measured bottom is 0.000230 m below the origin.
+    MiR1350_link.stl is a link-local derivative of the reduced 36,106-triangle
+    source mesh. Its metre scale, approved +pi/2 yaw, and 0.000230 m bottom
+    correction are baked into the vertices so every URDF viewer can use an
+    identity visual transform.
   -->
-  <xacro:property name="mir_stl_scale" value="1.0"/>
   <xacro:property name="mir_visual_length" value="1.350"/>
   <xacro:property name="mir_visual_width" value="0.910"/>
   <xacro:property name="mir_visual_height" value="0.321230"/>
-  <xacro:property name="mir_visual_bottom_offset" value="-0.000230"/>
-  <!-- Cancel the small negative STL minimum so the mesh bottom is at base_link. -->
-  <xacro:property name="mir_visual_z_offset" value="${-mir_visual_bottom_offset}"/>
-  <xacro:property name="mir_mesh_yaw" value="${pi / 2}"/>
   <!-- The 5 mm per-side collision clearance is deliberately conservative. -->
   <xacro:property name="chassis_length" value="1.340"/>
@@ -56,9 +51,8 @@
   <link name="base_link">
     <visual>
-      <origin xyz="0 0 ${mir_visual_z_offset}" rpy="0 0 ${mir_mesh_yaw}"/>
+      <origin xyz="0 0 0" rpy="0 0 0"/>
       <geometry>
-        <!-- The reduced mesh is already in metres. -->
-        <mesh filename="package://burke_description/cad/stl/MiR1350_reduced.stl"
-              scale="${mir_stl_scale} ${mir_stl_scale} ${mir_stl_scale}"/>
+        <mesh filename="package://burke_description/cad/stl/MiR1350_link.stl"
+              scale="1 1 1"/>
       </geometry>
       <material name="mir_gray"/>

File: burke_description/urdf/components/liftkit.urdf.xacro (robot description, xacro)
@@ -3,13 +3,10 @@
   <!--
     Three-stage LiftKit mast. The supplied STL files are millimetre CAD
-    exports in a common, fully extended assembly frame. Stage 1 is fixed to
-    the mobile base in this milestone; Task 3 will re-parent the arm to the
-    top stage.
+    exports in a common, fully extended assembly frame. The *_link.stl
+    derivatives bake their scale, orientation, and collapsed-stage offsets
+    into metre-scale vertices in each URDF link frame.
     All physical values below are simulation assumptions. The supplied CAD
     does not provide LiftKit mass properties or actuator ratings.
   -->
-  <xacro:property name="lift_mesh_scale" value="0.001"/>
-  <xacro:property name="lift_mesh_roll" value="${pi / 2}"/>
-  <xacro:property name="lift_mount_yaw" value="0.0"/>
   <!-- CAD-derived scaled envelopes, retained in named properties for review. -->
   <xacro:property name="stage_1_length" value="0.3229"/>
@@ -89,10 +86,8 @@
     <link name="lift_stage_1_link">
       <visual name="lift_stage_1_visual">
-        <!-- Keep the CAD centreline at raw x=0, z=0; do not centre its
-             asymmetric -X actuator housing AABB. -->
-        <origin xyz="0 0 0" rpy="${lift_mesh_roll} 0 ${lift_mount_yaw}"/>
+        <origin xyz="0 0 0" rpy="0 0 0"/>
         <geometry>
-          <mesh filename="package://burke_description/cad/stl/LIFTKIT_1.stl"
-                scale="${lift_mesh_scale} ${lift_mesh_scale} ${lift_mesh_scale}"/>
+          <mesh filename="package://burke_description/cad/stl/LIFTKIT_1_link.stl"
+                scale="1 1 1"/>
         </geometry>
         <material name="liftkit_gray"/>
@@ -114,9 +109,8 @@
     <link name="lift_stage_2_link">
       <visual name="lift_stage_2_visual">
-        <!-- Collapsed CAD retraction: -275 mm in the robot +Z frame. -->
-        <origin xyz="0 0 -0.275" rpy="${lift_mesh_roll} 0 0"/>
+        <origin xyz="0 0 0" rpy="0 0 0"/>
         <geometry>
-          <mesh filename="package://burke_description/cad/stl/LIFTKIT_2.stl"
-                scale="${lift_mesh_scale} ${lift_mesh_scale} ${lift_mesh_scale}"/>
+          <mesh filename="package://burke_description/cad/stl/LIFTKIT_2_link.stl"
+                scale="1 1 1"/>
         </geometry>
         <material name="liftkit_gray"/>
@@ -141,9 +135,8 @@
     <link name="lift_stage_3_link">
       <visual name="lift_stage_3_visual">
-        <!-- Collapsed CAD retraction: -500 mm absolute in the robot +Z frame. -->
-        <origin xyz="0 0 -0.500" rpy="${lift_mesh_roll} 0 0"/>
+        <origin xyz="0 0 0" rpy="0 0 0"/>
         <geometry>
-          <mesh filename="package://burke_description/cad/stl/LIFTKIT_3.stl"
-                scale="${lift_mesh_scale} ${lift_mesh_scale} ${lift_mesh_scale}"/>
+          <mesh filename="package://burke_description/cad/stl/LIFTKIT_3_link.stl"
+                scale="1 1 1"/>
         </geometry>
         <material name="liftkit_gray"/>

File: burke_description/urdf/components/ur8long.urdf.xacro (robot description, xacro)
@@ -3,5 +3,5 @@
   <!--
     UR8 Long arm using Universal Robots' official rolling configuration data.
-    The visual configuration points at the seven locally supplied STL parts;
+    The seven *_link.stl visual derivatives are metre-scale and link-local;
     collision geometry remains primitive for stable, inexpensive simulation.
   -->
@@ -28,7 +28,6 @@
     <xacro:macro name="mesh_visual" params="key">
       <xacro:property name="entry" value="${visual_data[key]}"/>
-      <xacro:property name="offset" value="${entry['mesh_offset']}"/>
       <visual>
-        <origin xyz="${offset['x']} ${offset['y']} ${offset['z']}" rpy="${offset['roll']} ${offset['pitch']} ${offset['yaw']}"/>
+        <origin xyz="0 0 0" rpy="0 0 0"/>
         <geometry>
           <mesh filename="package://burke_description/${entry['path']}" scale="${entry['scale']} ${entry['scale']} ${entry['scale']}"/>
